File: board/dmx-relay-puck.sch (EAGLE design)
At the start: 41 parts, among them J1 PJ-202A, J2 CON-3.81MM-1X6-PHOENIX-, J3 5520251-4, J4 5520251-4, J5 MOLEX-87758-1016, K1 G5V-1-5DC, K2 G5V-1-5DC, K3 G5V-1-5DC, K4 G5V-1-5DC, Q1 FMMT619TA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

Commit message: updated with notes on part substitutions and part stuffing
Other:
- note added: "FMMT619TA substitute: Fairchild/ON Semi #FSB619"
- note added: "Lower cost and more readily available substitute for 0.1µF 50V caps is Kemet #C1206C104K5RAC7867"
- note added: "MBR0580S1-7 substitute: Micro Commercial #MBR0580-TP"
- note added: "Notes: •replace R3 with 0Ω jumper •0Ω Bourns #CR1206-J/-000ELF •do not stuff C9"
Changed lines of the file:
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@@
 <text x="271.526" y="122.682" size="1.27" layer="91">MBR0580S1-7</text>
 <text x="368.3" y="227.838" size="1.778" layer="91">mates with 1803617</text>
+<text x="68.58" y="43.18" size="1.778" layer="97">Notes:
+•replace R3 with 0Ω jumper
+•0Ω Bourns #CR1206-J/-000ELF
+•do not stuff C9</text>
+<text x="134.62" y="15.24" size="1.778" layer="97">Lower cost and more readily available
+substitute for 0.1µF 50V caps is
+Kemet #C1206C104K5RAC7867</text>
+<text x="198.12" y="193.04" size="1.778" layer="97">FMMT619TA substitute:
+Fairchild/ON Semi #FSB619</text>
+<text x="198.12" y="185.42" size="1.778" layer="97">MBR0580S1-7 substitute:
+Micro Commercial #MBR0580-TP</text>
 </plain>
 <instances>
@@
 </schematic>
 </drawing>
+<compatibility>
+<note version="6.3" minversion="6.2.2" severity="warning">
+Since Version 6.2.2 text objects can contain more than one line,
+which will not be processed correctly with this version.
+</note>
+</compatibility>
 </eagle>
